Commit message: lidar fixed

File: turms_description/urdf/caster_wheel.xacro (robot description, xacro)
@@ -35,5 +35,6 @@
     </gazebo>
     <!-- CASTER WHEEL SUPPORT LINK -->
-    <joint name="caster_support_joint" type="continuous">
+    <!--joint name="caster_support_joint" type="continuous"-->
+    <joint name="caster_support_joint" type="fixed">
         <parent link="caster_base"/>
         <child link="caster_support"/>
@@ -65,5 +66,6 @@
     </gazebo>
     <!-- CASTER WHEEL LINK -->
-    <joint name="caster_wheel_joint" type="continuous">
+    <!--joint name="caster_wheel_joint" type="continuous"-->
+    <joint name="caster_wheel_joint" type="fixed">
         <parent link="caster_support"/>
         <child link="caster_wheel"/>

File: turms_description/urdf/lidar.xacro (robot description, xacro)
@@ -33,5 +33,5 @@
         <sensor name="laser" type="ray">
             <pose> 0 0 0 0 0 0 </pose>
-            <visualize>false</visualize>
+            <visualize>true</visualize>
             <update_rate>10</update_rate>
             <ray>

File: turms_description/urdf/lidar2d.xacro (robot description, xacro)
@@ -66,5 +66,5 @@
         <parent link="servo_stick_frame"/>
         <child link="ultrasonic_sensor_frame"/>
-        <origin xyz="0 0 ${servo_stick_heigth/2 + ultrasonic_sensor_heigth/2}" rpy="0 0 0"/>
+        <origin xyz="0 0 ${servo_stick_heigth/2 + ultrasonic_sensor_heigth/2}" rpy="0 0 ${pi}"/>
     </joint>
     <link name="ultrasonic_sensor_frame">
@@ -106,12 +106,12 @@
                 <scan>
                     <horizontal>
-                        <samples>1</samples>
-                        <min_angle>-3.14</min_angle>
-                        <max_angle>3.14</max_angle>
+                        <samples>2</samples>
+                        <min_angle>-0.01</min_angle>
+                        <max_angle>0.01</max_angle>
                     </horizontal>
                 </scan>
                 <range>
-                    <min>0.3</min>
-                    <max>12</max>
+                    <min>0.2</min>
+                    <max>50</max>
                 </range>
             </ray>
@@ -121,5 +121,5 @@
                 </ros>
                 <output_type>sensor_msgs/LaserScan</output_type>
-                <frame_name>laser_frame</frame_name>
+                <frame_name>ultrasonic_sensor_frame</frame_name>
             </plugin>
         </sensor>

File: turms_description/urdf/ros2_control.xacro (robot description, xacro)
@@ -59,8 +59,14 @@
                 <state_interface name="position"/>
             </joint>
+            <joint name="caster_support_joint">
+                <state_interface name="position"/>
+            </joint>
+            <joint name="caster_wheel_joint">
+                <state_interface name="position"/>
+            </joint>
             <joint name="servo_motor_joint">
                 <command_interface name="position">
-                    <param name="min">-1</param>
-                    <param name="max">1</param>
+                    <param name="min">-3.14</param>
+                    <param name="max">3.14</param>
                 </command_interface>
                 <state_interface name="position"/>

File: turms_ros2control/ros2_control/turms_ros2_control.xacro (robot description, xacro)
@@ -10,5 +10,5 @@
           <param name="right_wheel_name">rigth_wheel_joint</param>
           <param name="encoder_ticks">40</param>
-          <param name="servo_name">servo_joint</param>
+          <param name="servo_name">lidar_joint</param>
           <param name="loop_rate">3.0</param>
           <param name="baud_rate">576000</param>
@@ -39,5 +39,5 @@
         <state_interface name="velocity"/>
       </joint>
-      <joint name="${prefix}servo_joint">
+      <joint name="${prefix}servo_motor_joint">
         <command_interface name="position">
           <param name="min">-90</param>

Commit message: Update mesh file paths to use package syntax

File: turms_description/urdf/caster_wheel.xacro (robot description, xacro)
@@ -15,5 +15,5 @@
         <visual>
             <geometry>
-                <mesh filename="file:///$(find turms_description)/mesh/wheels/caster_base.stl" scale ="2 2 2"/>
+                <mesh filename="package://find turms_description/mesh/wheels/caster_base.stl" scale ="2 2 2"/>
                 <!--sphere radius="${caster_wheel_radius}"/-->
             </geometry>
@@ -45,5 +45,5 @@
             <origin xyz="0 0 -0.002" rpy="0 0 0" />
             <geometry>
-                <mesh filename="file:///$(find turms_description)/mesh/wheels/caster_wheel_support.stl" scale ="2 2 2"/>
+                <mesh filename="package://turms_description/mesh/wheels/caster_wheel_support.stl" scale ="2 2 2"/>
                 <!--sphere radius="${caster_wheel_radius}"/-->
             </geometry>
@@ -75,5 +75,5 @@
         <origin xyz="0 0 0" rpy="${pi/2} 0 0"/>
             <geometry>
-                <mesh filename="file:///$(find turms_description)/mesh/wheels/caster_wheel.stl" scale ="2 2 2"/>
+                <mesh filename="package://turms_description/mesh/wheels/caster_wheel.stl" scale ="2 2 2"/>
                 <!--sphere radius="${caster_wheel_radius}"/-->
             </geometry>
